File: GD32_SPINE.kicad_pcb (KiCad board)
At the start: 4 copper layers, 50 x 50 mm, 37 parts, among them J1 Barrel_Jack_MountingPin, J10 Conn_01x05, J11 Conn_01x02, J12 Conn_01x02, J2 Conn_01x08, J3 Conn_01x04, J4 Conn_01x03, J5 Conn_01x03, J6 Conn_01x10, J7 Conn_01x06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

Commit message: version 0.2
Parts:
- removed SW1: SW_Push, Connector_PinHeader_2.54mm:PinHeader_1x02_P2.54mm_Vertical
- added J13: Conn_ARM_JTAG_SWD_10, Connector_PinHeader_1.27mm:PinHeader_2x05_P1.27mm_Vertical, F.Cu at (108.3, 56.2)
- added J14: Conn_01x02, Connector_PinHeader_2.54mm:PinHeader_1x02_P2.54mm_Vertical, F.Cu at (111.8, 97.5)
- C1, C2: value 6.8pf -> 6.8pF; footprint Capacitor_SMD:C_0402_1005Metric -> Capacitor_SMD:C_0603_1608Metric_Pad1.08x0.95mm_HandSolder
- C3, C4: value 5.1pf -> 5.1pF; footprint Capacitor_SMD:C_0402_1005Metric -> Capacitor_SMD:C_0603_1608Metric_Pad1.08x0.95mm_HandSolder
- C5, C7: value 10uf -> 10uF; footprint Capacitor_SMD:C_0402_1005Metric -> Capacitor_SMD:C_1206_3216Metric_Pad1.33x1.80mm_HandSolder
- C6, C8: value 100nf -> 100nF; footprint Capacitor_SMD:C_0402_1005Metric -> Capacitor_SMD:C_0603_1608Metric_Pad1.08x0.95mm_HandSolder
- C9: footprint Capacitor_SMD:C_0402_1005Metric -> Capacitor_SMD:C_0603_1608Metric_Pad1.08x0.95mm_HandSolder
- J7: value Conn_01x06 -> Conn_01x02; footprint Connector_PinHeader_2.54mm:PinHeader_1x06_P2.54mm_Vertical -> Connector_PinHeader_2.54mm:PinHeader_1x02_P2.54mm_Vertical
- R1, R2, R3, R4, R5, R6, R7, R8, R9: footprint Resistor_SMD:R_0402_1005Metric -> Capacitor_SMD:C_0603_1608Metric_Pad1.08x0.95mm_HandSolder
- Y2: footprint Crystal:Crystal_SMD_3225-4Pin_3.2x2.5mm -> Crystal:Crystal_SMD_3215-2Pin_3.2x1.5mm
- moved R2 10.9 mm to (115.5, 90.5)
- moved R1 10.9 mm to (115.5, 88.5)
- moved C1 6.82 mm to (125.2, 75.0), turned to 90 degrees
- moved C2 6.79 mm to (125.2, 71.0), turned to -90 degrees
- moved C3 5.22 mm to (127.0, 81.0), turned to 90 degrees
- moved C4 5.00 mm to (127.0, 77.2), turned to -90 degrees
- moved C6 4.61 mm to (135.0, 70.2), turned to 90 degrees
- moved R8 4.07 mm to (127.0, 88.5)
- moved R9 3.58 mm to (127.0, 90.5)
- moved C8 3.25 mm to (135.0, 77.2), turned to 90 degrees
- moved R7 3.25 mm to (108.8, 62.0)
- moved U3 2.50 mm to (122.0, 90.0)
- moved C9 2.47 mm to (106.8, 62.0)
- moved C5 1.90 mm to (137.8, 69.5), turned to 90 degrees
- moved R3 1.64 mm to (134.7, 82.0)
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Connections:
- J6 pad 5: USART2_TX -> USART1_TX
- J6 pad 6: USART2_RX -> USART1_RX
- J6 pad 8: USART1_TX -> USART2_TX
- J6 pad 9: USART1_RX -> USART2_RX
- Y2 pad 2: GND -> Net-(C3-Pad2)
Routing:
- net Net-(R2-Pad2): track 14.3 -> 3.92 mm
- net Net-(R1-Pad2): track 18.7 -> 9.02 mm
- net SWCLK: track 31.4 -> 40.5 mm
- net I2C0_SDA: track 37.0 -> 29.3 mm
- net I2C0_SCL: track 41.8 -> 34.2 mm
- net USART0_RX: track 45.1 -> 37.9 mm
- net USART0_TX: track 47.6 -> 40.4 mm
- net SWDIO: track 29.5 -> 35.6 mm
- net GND: track 14.4 -> 20.0 mm, vias 105 -> 119
- net Net-(C2-Pad2): track 14.0 -> 8.79 mm
- net USART2_TX: track 18.4 -> 14.1 mm
- net PA15: track 23.1 -> 26.8 mm
- net USART2_RX: track 17.5 -> 14.1 mm
- net Net-(C4-Pad2): track 13.4 -> 10.0 mm
- net Net-(C1-Pad2): track 13.6 -> 10.3 mm
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- added copper zone on In2.Cu, net +12V
Other:
- board text added: "GD32 SPINE By Ashlee Nov 26, 2021 Version 0.2"
- board text removed: "GD32 SPINE By Ashlee Oct 23, 2021 Version 0.1"
