File: GD32_SPINE.kicad_sch (KiCad schematic)
At the start: 37 parts, among them J1 Barrel_Jack_MountingPin, J10 Conn_01x05, J11 Conn_01x02, J12 Conn_01x02, J2 Conn_01x08, J3 Conn_01x04, J4 Conn_01x03, J5 Conn_01x03, J6 Conn_01x10, J7 Conn_01x06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

Commit message: version 0.2
Parts:
- removed J7: Conn_01x06, Connector_PinHeader_2.54mm:PinHeader_1x06_P2.54mm_Vertical, symbol Connector_Generic:Conn_01x06
- removed SW1: SW_Push, Connector_PinHeader_2.54mm:PinHeader_1x02_P2.54mm_Vertical, symbol Switch:SW_Push
- added J13: Conn_ARM_JTAG_SWD_10, Connector_PinHeader_1.27mm:PinHeader_2x05_P1.27mm_Vertical, symbol Connector:Conn_ARM_JTAG_SWD_10
- added J14, J7: Conn_01x02, Connector_PinHeader_2.54mm:PinHeader_1x02_P2.54mm_Vertical, symbol Connector_Generic:Conn_01x02
- C1, C2: value 6.8pf -> 6.8pF; footprint Capacitor_SMD:C_0402_1005Metric -> Capacitor_SMD:C_0603_1608Metric_Pad1.08x0.95mm_HandSolder
- C3, C4: value 5.1pf -> 5.1pF; footprint Capacitor_SMD:C_0402_1005Metric -> Capacitor_SMD:C_0603_1608Metric_Pad1.08x0.95mm_HandSolder
- C5, C7: value 10uf -> 10uF; footprint Capacitor_SMD:C_0402_1005Metric -> Capacitor_SMD:C_1206_3216Metric_Pad1.33x1.80mm_HandSolder
- C6, C8: value 100nf -> 100nF; footprint Capacitor_SMD:C_0402_1005Metric -> Capacitor_SMD:C_0603_1608Metric_Pad1.08x0.95mm_HandSolder
- C9: footprint Capacitor_SMD:C_0402_1005Metric -> Capacitor_SMD:C_0603_1608Metric_Pad1.08x0.95mm_HandSolder
- R1, R2, R3, R4, R5, R6, R7, R8, R9: footprint Resistor_SMD:R_0402_1005Metric -> Capacitor_SMD:C_0603_1608Metric_Pad1.08x0.95mm_HandSolder
- Y2: footprint Crystal:Crystal_SMD_3225-4Pin_3.2x2.5mm -> Crystal:Crystal_SMD_3215-2Pin_3.2x1.5mm; symbol Device:Crystal_GND24_Small -> Device:Crystal_Small
Connections:
- net +3V3: now also J13.1 (VTref)
- net CAN0_H: now also J7.1 (Pin_1)
- net CAN0_L: now also J7.2 (Pin_2)
- net CAN1_H: now also J14.1 (Pin_1)
- net CAN1_L: now also J14.2 (Pin_2)
- net GND: now also J13.3 (GND), J13.5 (GND), J13.9 (GNDDetect); no longer Y2.2, Y2.4
- net NRST: now also J13.10 (~{RESET})
- net SWCLK: now also J13.4 (SWDCLK/TCK)
- net SWDIO: now also J13.2 (SWDIO/TMS)
- net USART1_RX: now also J6.6 (Pin_6); no longer J6.9 (Pin_9)
- net USART1_TX: now also J6.5 (Pin_5); no longer J6.8 (Pin_8)
- net USART2_RX: now also J6.9 (Pin_9); no longer J6.6 (Pin_6)
- net USART2_TX: now also J6.8 (Pin_8); no longer J6.5 (Pin_5)
- net at C3.2, U1.3 (PC14): now also Y2.2; no longer Y2.3
- no-connect marks 1 -> 3
